File: op6-jig.sch (KiCad schematic (older format))
At the start: 43 parts, among them J1 PHONE_TP_BREAKOUT, J2 JTAG_ATMEGA, J3 ATMEGA_MISC_GPIO, P1 USB_C_ATMEGA, P2 USB_C_PHONE, Q1 FQP27P06, SW1 SW_RESET, U1 ATMEGA32U4, U2 LSF0102YZTR, Y1 16MHz

Commit message: pcb: rewire by hand
hah, i actually did it...

The PCB is now hand wired and muuuuuuuch better. This drops the USB pins
on the breakout header because they probably aren't needed and added too
much complexity to the traces.

Also replace the UART pinout with the 5v one on the Atmega side of the
level shifter rather than the 1.8v levels at the phone.
 * This would mean UART is borked unless you attach 5v to the Atmega USB
   port, maybe we want to power the level shifter with the phone vbus
   supply instead ?
Parts:
- C1, C2, C3, C4, C5, C6, C7: symbol Device:C_Small -> op6-jig-rescue:C_Small-Device
- D1, D2, D3: symbol Device:LED -> op6-jig-rescue:LED-Device
- H1, H10, H11, H12, H13, H2, H3, H6, H7, H8, H9: symbol Connector:TestPoint_Probe -> op6-jig-rescue:TestPoint_Probe-Connector
- H4: value PHONE_USB_DN -> PHONE_USB_D-; symbol Connector:TestPoint_Probe -> op6-jig-rescue:TestPoint_Probe-Connector
- H5: value PHONE_USB_DP -> PHONE_USB_D+; symbol Connector:TestPoint_Probe -> op6-jig-rescue:TestPoint_Probe-Connector
- J1: symbol Connector_Generic:Conn_02x10_Counter_Clockwise -> op6-jig-rescue:Conn_02x10_Counter_Clockwise-Connector_Generic
- J2: symbol Connector_Generic:Conn_02x05_Odd_Even -> op6-jig-rescue:Conn_02x05_Odd_Even-Connector_Generic
- J3: symbol Connector_Generic:Conn_01x04 -> op6-jig-rescue:Conn_01x04-Connector_Generic
- Q1: symbol Transistor_FET:FQP27P06 -> op6-jig-rescue:FQP27P06-Transistor_FET
- R10, R11, R12, R3, R4, R5, R6, R7, R8, R9: symbol Device:R -> op6-jig-rescue:R-Device
- SW1: symbol Switch:SW_Push -> op6-jig-rescue:SW_Push-Switch
- U1: symbol ATmega32U4:ATMEGA32U4 -> op6-jig-rescue:ATMEGA32U4-ATmega32U4
- Y1: symbol Device:Crystal -> op6-jig-rescue:Crystal-Device
Connections:
- net GND: now also J1.19 (Pin_19); no longer J1.20 (Pin_20)
- net PHONE_RX: no longer J1.19 (Pin_19)
- net PHONE_TX: no longer J1.18 (Pin_18)
- net PHONE_USB_CC: no longer J1.7 (Pin_7)
- net ATMEGA_USB_D-: now reaches P1.A6 (D+), P1.B6 (D+), R5.2
- net ATMEGA_USB_D+: now reaches P1.A7 (D-), P1.B7 (D-), R6.2
- net LEG_B_EN: now reaches R11.2, U1.10 (PB2)
- net ATMEGA_RX: now reaches U1.20 (PD2), U2.3 (A1)
- net ATMEGA_RX: now also J1.20 (Pin_20)
- net ATMEGA_TX: now reaches U1.21 (PD3), U2.4 (A2)
- net ATMEGA_TX: now also J1.18 (Pin_18)
- net ATMEGA_USB_R_D+: now reaches R6.1, U1.3 (D-)
- net at U1.31 (PC6): now also J3.2 (Pin_2); no longer J3.1 (Pin_1)
- net at U1.32 (PC7): now also J3.1 (Pin_1); no longer J3.2 (Pin_2)
- net ATMEGA_USB_R_D-: now reaches R5.1, U1.4 (D+)
- net LED_R_EN: now reaches R9.2, U1.8 (PB0)
- net LED_G_EN: now reaches R10.2, U1.9 (PB1)
- net PHONE_USB_DN renamed PHONE_USB_D-
- net PHONE_USB_D-: no longer J1.5 (Pin_5)
- net PHONE_USB_DP renamed PHONE_USB_D+
- net PHONE_USB_D+: no longer J1.6 (Pin_6)

Commit message: updates, ready-er to produce?
* Replaced the mosfet with a switching IC (thanks @A13).
* Removed ATMEGA MISC header, put those pins on the general 20-pin
  header.
* Replaced USB-C part with a better SMD part (thanks again @A13).
* Some misc fixes / routing improvements.
Parts:
- removed J3: ATMEGA_MISC_GPIO, Connector_PinHeader_2.54mm:PinHeader_1x04_P2.54mm_Vertical, symbol op6-jig-rescue:Conn_01x04-Connector_Generic
- removed P1: USB_C_ATMEGA, Connector_USB:USB_C_Receptacle_GCT_USB4085, symbol custom-symbols:USB_C_Plug_USB2.0_bidirectional
- removed P2: USB_C_PHONE, Connector_USB:USB_C_Receptacle_GCT_USB4085, symbol custom-symbols:USB_C_Plug_USB2.0_bidirectional
- removed Q1: FQP27P06, Package_TO_SOT_THT:TO-220-3_Vertical, symbol op6-jig-rescue:FQP27P06-Transistor_FET
- removed R12: 10k, Resistor_SMD:R_0805_2012Metric_Pad1.20x1.40mm_HandSolder, symbol op6-jig-rescue:R-Device
- added J4, J5: TYPE-C-31-M-12, Local:HRO_TYPE-C-31-M-12, symbol HRO_TYPE-C:TYPE-C-31-M-12
- added R1, R2: 5.1k, Resistor_SMD:R_0805_2012Metric_Pad1.20x1.40mm_HandSolder, symbol op6-jig-rescue:R-Device
- added U3: AP2192, Package_SO:SO-8_3.9x4.9mm_P1.27mm, symbol kicad-open-libs:AP2192-on-grid
- C1, C4: LCSC (none) -> C28323
- C2, C3: LCSC (none) -> C1804
- C5, C6, C7: value 0.1uF -> 100nF; LCSC (none) -> C49678
- D1: LCSC (none) -> C84256
- D2, D3: LCSC (none) -> C2297
- R10, R11, R9: LCSC (none) -> C17557
- R3: LCSC (none) -> C26010
- R4, R7: LCSC (none) -> C22859
- R5, R6: LCSC (none) -> C17561
- R8: value 5k -> 5.6k; LCSC (none) -> C4382
- U2: LCSC (none) -> C132024
Connections:
- net 5v: now also J4.A4B9 (VBUS), J4.B4A9 (VBUS)
- net ATMEGA_USB_D+: now also J4.A6 (DP1), J4.B6 (DP2)
- net ATMEGA_USB_D-: now also J4.A7 (DN1), J4.B7 (DN2)
- net GND: now also J4.A1B12 (GND), J4.B1A12 (GND), J4.S1 (SHIELD), J4.S2 (SHIELD), J4.S3 (SHIELD), J4.S4 (SHIELD), J5.A1B12 (GND), J5.B1A12 (GND), J5.S1 (SHIELD), J5.S2 (SHIELD), J5.S3 (SHIELD), J5.S4 (SHIELD), R1.2, R2.2, U3.1 (GND)
- net PHONE_USB_CC: now also J5.A5 (CC1), J5.B5 (CC2)
- net PHONE_USB_D+: now also J5.A6 (DP1), J5.B6 (DP2)
- net PHONE_USB_D-: now also J5.A7 (DN1), J5.B7 (DN2)
- net PHONE_VBUS: now also J5.A4B9 (VBUS), J5.B4A9 (VBUS), U3.2 (IN)
- net PHONE_VBUS_SWITCHED: now also U3.7 (OUT1)
- net VBUS_EN: now also U3.3 (EN1)
- net ATMEGA_PD0: now reaches U1.18 (PD0)
- net ATMEGA_PD0: now also J1.5 (Pin_5)
- net ATMEGA_PD1: now reaches U1.19 (PD1)
- net ATMEGA_PD1: now also J1.4 (Pin_4)
- net AP_VBUS_FAULT1: now reaches U1.26 (PD6)
- net AP_VBUS_FAULT1: now also U3.8 (FLG1)
- net ATMEGA_PC6: now reaches U1.31 (PC6)
- net ATMEGA_PC6: now also J1.7 (Pin_7)
- net ATMEGA_PC7: now reaches U1.32 (PC7)
- net ATMEGA_PC7: now also J1.6 (Pin_6)
- new net: J4.A5 (CC1), R1.1
- new net: J4.B5 (CC2), R2.1
- no-connect marks 12 -> 14
Other:
- note added: "Pull up"

Commit message: Final-final-v2.docx (it's ordered)
- Replaced the precisely positioned and probably wrong test points with
  a pin header connector which can just be soldered too.
- Cleaned up some traces, resized all vias to be a minimum of 0.45mm for
  JLCPCB.
- Ordered the board!
Parts:
- removed H1: Rx, op6-jig:TestPoint_Plated_Hole_D0.9mm, symbol op6-jig-rescue:TestPoint_Probe-Connector
- removed H10: PWR_BTN, op6-jig:TestPoint_Plated_Hole_D0.9mm, symbol op6-jig-rescue:TestPoint_Probe-Connector
- removed H11: BOOT_MODE_0, op6-jig:TestPoint_Plated_Hole_D0.9mm, symbol op6-jig-rescue:TestPoint_Probe-Connector
- removed H12: BOOT_MODE_1, op6-jig:TestPoint_Plated_Hole_D0.9mm, symbol op6-jig-rescue:TestPoint_Probe-Connector
- removed H13: GND, op6-jig:TestPoint_Plated_Hole_D0.9mm, symbol op6-jig-rescue:TestPoint_Probe-Connector
- removed H2: Tx, op6-jig:TestPoint_Plated_Hole_D0.9mm, symbol op6-jig-rescue:TestPoint_Probe-Connector
- removed H3: PHONE_VBUS, op6-jig:TestPoint_Plated_Hole_D0.9mm, symbol op6-jig-rescue:TestPoint_Probe-Connector
- removed H4: PHONE_USB_D-, op6-jig:TestPoint_Plated_Hole_D0.9mm, symbol op6-jig-rescue:TestPoint_Probe-Connector
- removed H5: PHONE_USB_D+, op6-jig:TestPoint_Plated_Hole_D0.9mm, symbol op6-jig-rescue:TestPoint_Probe-Connector
- removed H6: PHONE_USB_CC, op6-jig:TestPoint_Plated_Hole_D0.9mm, symbol op6-jig-rescue:TestPoint_Probe-Connector
- removed H7: VBAT0, op6-jig:TestPoint_Plated_Hole_D0.9mm, symbol op6-jig-rescue:TestPoint_Probe-Connector
- removed H8: VOL_DOWN, op6-jig:TestPoint_Plated_Hole_D0.9mm, symbol op6-jig-rescue:TestPoint_Probe-Connector
- removed H9: VOL_UP, op6-jig:TestPoint_Plated_Hole_D0.9mm, symbol op6-jig-rescue:TestPoint_Probe-Connector
- added J3: CONN_PHONE_DATA, Connector_PinHeader_2.54mm:PinHeader_1x10_P2.54mm_Vertical, symbol Connector_Generic:Conn_01x10
- added J6: CONN_PHONE_POWER, Connector_PinHeader_2.54mm:PinHeader_1x03_P2.54mm_Vertical, symbol Connector_Generic:Conn_01x03
- C1, C2, C3, C4, C5, C6, C7: footprint Capacitor_SMD:C_0805_2012Metric_Pad1.18x1.45mm_HandSolder -> Capacitor_SMD:C_0805_2012Metric
- J1: footprint Connector_PinHeader_2.54mm:PinHeader_2x10_P2.54mm_Horizontal -> Connector_PinHeader_2.54mm:PinHeader_2x10_P2.54mm_Vertical
- R1, R10, R11, R2, R3, R4, R5, R6, R7, R8, R9: footprint Resistor_SMD:R_0805_2012Metric_Pad1.20x1.40mm_HandSolder -> Resistor_SMD:R_0805_2012Metric
Connections:
- net BOOT_MODE_0: now also J3.5 (Pin_5)
- net BOOT_MODE_1: now also J3.4 (Pin_4)
- net GND: now also J6.2 (Pin_2)
- net PHONE_RX: now also J3.8 (Pin_8)
- net PHONE_TX: now also J3.7 (Pin_7)
- net PHONE_USB_CC: now also J3.3 (Pin_3)
- net PHONE_USB_D+: now also J3.2 (Pin_2)
- net PHONE_USB_D-: now also J3.1 (Pin_1)
- net PHONE_VBUS_SWITCHED: now also J6.1 (Pin_1)
- net PWR_BTN: now also J3.6 (Pin_6)
- net VBAT: now also J6.3 (Pin_3)
- net VOL_DOWN: now also J3.10 (Pin_10)
- net VOL_UP: now also J3.9 (Pin_9)

Commit message: uhhh
Parts:
- U1: footprint ATmega32U4:ATmega32U4 -> Atmega32u4:ATmega32U4
Changed lines of the file:
@@
 F 0 "U1" H 5400 3820 50  0000 C CNN
 F 1 "ATMEGA32U4" H 5400 3729 50  0000 C CNN
-F 2 "ATmega32U4:ATmega32U4" H 5350 3650 50  0001 L BNN
+F 2 "Atmega32u4:ATmega32U4" H 5350 3650 50  0001 L BNN
 F 3 "" H 5100 3850 50  0001 L BNN
 	1    5400 2350
